Commit message: Fix wheel joint origins and add wheel visuals

File: description/robot_core.xacro (robot description, xacro)
@@ -32,5 +32,5 @@
         <parent link="base_link"/>
         <child link="left_wheel"/>
-        <origin xyz="0 0.175 0 rpy="-${pi/2}" 0 0"/>
+        <origin xyz="0 0.175 0" rpy="-${pi/2}" 0 0"/>
 <axis xyz="0 0 1"/>
 </joint>
@@ -47,5 +47,5 @@
         <parent link="base_link"/>
         <child link="right_wheel"/>
-        <origin xyz="0 -0.175 0 rpy="-${pi/2}" 0 0"/>
+        <origin xyz="0 -0.175 0" rpy="-${pi/2}" 0 0"/>
         <axis xyz="0 0 1"/>
     </joint>

Commit message: REattempt ot fix joint state

File: description/robot_core.xacro (robot description, xacro)
@@ -30,31 +30,31 @@
 <!-- LEFT WHEEL LINK -->
 <joint name="left_wheel_joint" type="continuous">
-        <parent link="base_link"/>
-        <child link="left_wheel"/>
-        <origin xyz="0 0.175 0" rpy="-${pi/2}" 0 0"/>
-<axis xyz="0 0 1"/>
+    <parent link="base_link"/>
+    <child link="left_wheel"/>
+    <origin xyz="0 0.175 0" rpy="-1.5708 0 0"/>
+    <axis xyz="0 0 1"/>
 </joint>
 <link name="left_wheel">
-        <visual>
-           <geometry>
-                <cylinder radius="0.05" length="0.04"/>
-            </geometry>
-            <material name="blue"/>
-        </visual>
-        </link>
+    <visual>
+        <geometry>
+            <cylinder radius="0.05" length="0.04"/>
+        </geometry>
+        <material name="blue"/>
+    </visual>
+</link>
 <!-- RIGHT WHEEL LINK -->
-    <joint name="right_wheel_joint" type="continuous">
-        <parent link="base_link"/>
-        <child link="right_wheel"/>
-        <origin xyz="0 -0.175 0" rpy="-${pi/2}" 0 0"/>
-        <axis xyz="0 0 1"/>
-    </joint>
-    <link name="right_wheel">
-        <visual>
-            <geometry>
-                <cylinder radius="0.05" length="0.04"/>
-            </geometry>
-            <material name="blue"/>
-        </visual>
-    </link>
+<joint name="right_wheel_joint" type="continuous">
+    <parent link="base_link"/>
+    <child link="right_wheel"/>
+    <origin xyz="0 -0.175 0" rpy="-1.5708 0 0"/>
+    <axis xyz="0 0 1"/>
+</joint>
+<link name="right_wheel">
+    <visual>
+        <geometry>
+            <cylinder radius="0.05" length="0.04"/>
+        </geometry>
+        <material name="blue"/>
+    </visual>
+</link>
 </robot>

Commit message: Caster Wheel Link

File: description/robot_core.xacro (robot description, xacro)
@@ -58,3 +58,17 @@
     </visual>
 </link>
+<!-- Caster Wheel link-->
+<joint name="caster_wheel_joint" type="fixed">
+    <parent link="chassis"/>
+    <child link="caster_wheel"/>
+    <origin xyz="0.24 0 0"/>
+    </joint>
+    <link name="caster_wheel">
+        <visual>
+            <geometry>
+             <sphere radius="0.05"/>
+            </geometry>
+            <material name="black"/>
+        </visual>
+    </link>
 </robot>

Commit message: Collision Added

File: description/robot_core.xacro (robot description, xacro)
@@ -27,5 +27,12 @@
             <material name="white"/>
         </visual>
+        <collision>
+            <origin xyz="0.15 0 0.075"/>
+            <geometry>
+                <box size="0.3 0.3 0.15"/>
+            </geometry>
+        </collision>
     </link>
+<!-- CHASSIS LINK END -->
 <!-- LEFT WHEEL LINK -->
 <joint name="left_wheel_joint" type="continuous">
@@ -42,4 +49,9 @@
         <material name="blue"/>
     </visual>
+    <collision>
+        <geometry>
+            <cylinder radius="0.05" length="0.04"/>
+        </geometry>
+    </collision>
 </link>
 <!-- RIGHT WHEEL LINK -->
@@ -57,4 +69,9 @@
         <material name="blue"/>
     </visual>
+      <collision>
+        <geometry>
+            <cylinder radius="0.05" length="0.04"/>
+        </geometry>
+    </collision>
 </link>
 <!-- Caster Wheel link-->
@@ -71,4 +88,9 @@
             <material name="black"/>
         </visual>
+           <collision>
+            <geometry>
+             <sphere radius="0.05"/>
+            </geometry>
+        </collision>
     </link>
 </robot>

Commit message: Adding collision

File: description/robot_core.xacro (robot description, xacro)
@@ -1,4 +1,5 @@
 <?xml version="1.0"?>
 <robot xmlns:xacro="http://www.ros.org/wiki/xacro">
+<xacro:include filename="inertial macros.xacro"/>
     <material name="white">
         <color rgba="1 1 1 1"/>
@@ -33,4 +34,7 @@
             </geometry>
         </collision>
+        <xacro:inertial_box mass="0.5" x="0.3" y="0.3" z="0.15" >
+            <origin xyz="0.15 0 0.075" rpy="0 0 0"/>
+        </xacro:inertial_box>
     </link>
 <!-- CHASSIS LINK END -->
@@ -54,4 +58,6 @@
         </geometry>
     </collision>
+    <xacro:inertial_cylinder mass="0.1" radius="0.05" length="0.04">
+        <origin xyz="0 0 0" rpy="0 0 0"/>
 </link>
 <!-- RIGHT WHEEL LINK -->
@@ -74,4 +80,6 @@
         </geometry>
     </collision>
+    <xacro:inertial_cylinder mass="0.1" radius="0.05" length="0.04">
+        <origin xyz="0 0 0" rpy="0 0 0"/>
 </link>
 <!-- Caster Wheel link-->
@@ -93,4 +101,6 @@
             </geometry>
         </collision>
+        <xacro:inertial_sphere mass="0.1" radius="0.05">
+            <origin xyz="0 0 0" rpy="0 0 0"/>
     </link>
 </robot>

Commit message: Defintion Clean up

File: description/robot_core.xacro (robot description, xacro)
@@ -10,4 +10,7 @@
     <material name="black">
         <color rgba="0 0 0 1"/>
+    </material>
+    <material name="blue">
+        <color rgba="0 0 1 1"/>
     </material>
 <!--BASE LINK -->
@@ -60,4 +63,5 @@
     <xacro:inertial_cylinder mass="0.1" radius="0.05" length="0.04">
         <origin xyz="0 0 0" rpy="0 0 0"/>
+        </xacro:inertial_cylinder>
 </link>
 <!-- RIGHT WHEEL LINK -->
@@ -82,4 +86,5 @@
     <xacro:inertial_cylinder mass="0.1" radius="0.05" length="0.04">
         <origin xyz="0 0 0" rpy="0 0 0"/>
+        </xacro:inertial_cylinder>
 </link>
 <!-- Caster Wheel link-->
@@ -103,4 +108,5 @@
         <xacro:inertial_sphere mass="0.1" radius="0.05">
             <origin xyz="0 0 0" rpy="0 0 0"/>
+        </xacro:inertial_sphere>
     </link>
 </robot>
